File: v4/FINAL VERSION/KiCad/final version.kicad_pcb (KiCad board)
At the start: 2 copper layers, 199.5 x 256 mm, 83 parts, among them J1 Raspberry_Pi_4, J2 Conn_01x04_Pin, J3 Conn_01x08_Pin, J4 AudioJack3, J5 Conn_01x04_Pin, U17 CD74HC4067M, U18 MCP3008, U19 PCM5102A, U20 TPA6132A2RTE, U21 SN74LV4052ADR

Commit message: update of PCB
Parts:
- C1, C10, C11, C12, C13, C14, C15, C16, C17, C18, C19, C2, C20, C21, C3, C4, C5, C6, C7, C8, C9: footprint Capacitor_SMD:C_0402_1005Metric_Pad0.74x0.62mm_HandSolder -> Capacitor_SMD:C_0805_2012Metric_Pad1.18x1.45mm_HandSolder
- R1, R10, R11, R12, R13, R14, R15, R16, R17, R18, R19, R2, R3, R4, R5, R6, R7, R8, R9: footprint Resistor_SMD:R_0402_1005Metric_Pad0.72x0.64mm_HandSolder -> Resistor_SMD:R_0805_2012Metric_Pad1.20x1.40mm_HandSolder
- moved U21 168.0 mm to (225.6, 102.3)
- moved U17 165.8 mm to (225.7, 117.9), turned to 180 degrees
- moved C1 150.9 mm to (217.3, 124.2), turned to 180 degrees
- moved C7 3.18 mm to (183.9, 70.8)
- moved C12 2.06 mm to (203.7, 74.0)
- moved C14 1.75 mm to (199.9, 81.0)
- moved C11 1.58 mm to (203.7, 70.0)
- moved C9 1.47 mm to (201.4, 73.9)
- moved C6 1.32 mm to (188.4, 70.3)
- moved C13 1.29 mm to (199.8, 78.4)
- moved R18 1.24 mm to (195.7, 81.0)
- moved C4 1.15 mm to (188.7, 76.8)
- moved C15 0.86 mm to (209.7, 75.3)
- moved C21 0.85 mm to (65.1, 146.2)
- moved C5 0.84 mm to (190.8, 70.3)
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Routing:
- net /MATRIX/7: track 319.1 -> 123.2 mm
- net /Rasp Pi/RX0: track 135.9 -> 329.7 mm, vias 1 -> 2
- net /MATRIX/6: track 364.2 -> 174.9 mm
- net /MATRIX/0: track 66.7 -> 253.4 mm, vias 0 -> 2
- net /MATRIX/1: track 117.5 -> 301.6 mm
- net /MATRIX/5: track 408.6 -> 225.8 mm
- net /MATRIX/2: track 168.9 -> 349.8 mm
- net /MATRIX/3: track 220.2 -> 397.9 mm
- net /MATRIX/4: track 452.0 -> 276.9 mm
- net /Rasp Pi/TX0: track 143.6 -> 318.2 mm, vias 1 -> 2
- net /MATRIX/12: track 550.5 -> 376.5 mm
- net /MATRIX/13: track 499.0 -> 331.7 mm
- net /Rasp Pi/TX1: track 296.0 -> 131.8 mm, vias 1 -> 0
- net /Rasp Pi/RX1: track 296.2 -> 133.8 mm, vias 1 -> 0
- net /MATRIX/14: track 447.3 -> 287.3 mm
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Other:
- board size 199.5 x 256 mm -> 199.5 x 256.1 mm
